File: 250407_.kicad_pcb (KiCad board)
At the start: 2 copper layers, 390 x 179.8 mm, 227 parts, among them CN1 KEYBOARD_20PIN_MALE, CN10 LED_CONNECTOR, CN2 USER_PORT_CON, CN3 CASSETTE_PORT_CON, CN4 SERIAL_BUS_CON, CN5 AV_CONN, CN6 EXPANSION_PORT, CN7 POWER_CON, CN8 CONTROL_PORT, CN9 CONTROL_PORT, M1 MODULATOR_LONGBOARD, Q1 2SC1815, Q2 2SC1815, Q3 TP29B/2SD880, Q7 2SC1815, Q8 2SC1815, SW1 POWER_SWITCH, U1 CIA_U1, U10 4164-2, U11 4164-2, U12 4164-2, U13 74LS257, U14 74LS258, U15 74LS139, U16 4066_U28, U17 PLA_U17, U18 6581, U19 VIC, U2 CIA_U2, U20 556, U21 4164-2, U22 4164-2, U23 4164-2, U24 4164-2, U25 74LS257, U26 74LS373, U27 7408_U27, U28 4066_U28, U29 74LS74, U3 2364A, U30 74LS193, U31 74LS629N, U32 MC4044, U4 2364A, U5 2332A, U6 2114, U7 6510_MPU, U8 7406N, U9 4164-2, Y1 Crystal

Commit message: V1.3. PAL-NTSC E1 E2 E3 fix. Saved in KiCAD 9.0.1
Parts:
- renumbered E1 to E3
Connections:
- net /'9VAC~~ renamed /'9VAC~
- net /250407_sheet2/GR\~W~ renamed /250407_sheet2/GR\~{W}
- net /250407_sheet2/~AEC~ renamed /250407_sheet2/~{AEC}
- net /250407_sheet2/~BASIC~ renamed /250407_sheet2/~{BASIC}
- net /250407_sheet2/~CASRAM~ renamed /250407_sheet2/~{CASRAM}
- net /250407_sheet2/~CASRAM~' renamed /250407_sheet2/~{CASRAM}'
- net /250407_sheet2/~CAS~ renamed /250407_sheet2/~{CAS}
- net /250407_sheet2/~CHAROM~ renamed /250407_sheet2/~{CHAROM}
- net /250407_sheet2/~CIAS~ renamed /250407_sheet2/~{CIAS}
- net /250407_sheet2/~COLOR~ renamed /250407_sheet2/~{COLOR}
- net /250407_sheet2/~DMA~ renamed /250407_sheet2/~{DMA}
- net /250407_sheet2/~EXROM~ renamed /250407_sheet2/~{EXROM}
- net /250407_sheet2/~GAME~ renamed /250407_sheet2/~{GAME}
- net /250407_sheet2/~I\O~ renamed /250407_sheet2/~{I\O}
- net /250407_sheet2/~KERNAL renamed /250407_sheet2/~{KERNAL}
- net /250407_sheet2/~RAS~ renamed /250407_sheet2/~{RAS}
- net /250407_sheet2/~RESET'~ renamed /250407_sheet2/~{RESET'}
- net /250407_sheet2/~ROMH~ renamed /250407_sheet2/~{ROMH}
- net /250407_sheet2/~ROML~ renamed /250407_sheet2/~{ROML}
- net /250407_sheet2/~SID~ renamed /250407_sheet2/~{SID}
- net /250407_sheet2/~VIC~ renamed /250407_sheet2/~{VIC}
- net /9VAC~~ renamed /9VAC~
- net /~FLAG2~ renamed /~{FLAG2}
- net /~PC2~ renamed /~{PC2}
- net /~RESTORE~ renamed /~{RESTORE}
- net BTNA\~LP~ renamed BTNA\~{LP}
- net R\~W~ renamed R\~{W}
- net ~CHAREN~ renamed ~{CHAREN}
- net ~CIA1~ renamed ~{CIA1}
- net ~CIA2~ renamed ~{CIA2}
- net ~HIRAM~ renamed ~{HIRAM}
- net ~IRQ~ renamed ~{IRQ}
- net ~LORAM~ renamed ~{LORAM}
- net ~NMI~ renamed ~{NMI}
- net ~RESET~ renamed ~{RESET}
- net ~VA14~ renamed ~{VA14}
- net ~VA15~ renamed ~{VA15}
Other:
- net class Default removed
- rule pad_to_mask_clearance: 0.051 -> 0
- board text added: "E1"
- board text added: "Replica ${REVISION} by BWACK 2021"
- board text removed: "Replica 1.1 by BWACK 2021"
